Commit message: update

File: i608_moveit_config/config/i608.ros2_control.xacro (robot description, xacro)
@@ -2,5 +2,59 @@
 <robot xmlns:xacro="http://www.ros.org/wiki/xacro" name="i608">
 	<xacro:macro name="i608_ros2_control" params="name initial_position_file">
-		<xacro:property name="initial_positions" value="${load_yaml(initial_positions_file)['initial_positions']}"></xacro:property>
+		<xacro:property name="initial_positions" value="${load_yaml(initial_positions_file)['initial_positions']}">
+			<ros2_control name="${name}" type="system">
+				<hardware>
+					<plugin>icnc_hardware_interfaces/I608SystemHardware</plugin>
+				</hardware>
+				<joint name="joint_1">
+					<command_interface name="position"></command_interface>
+					<command_interface name="velocity"></command_interface>
+					<state_interface name="position">
+						<param name="initial_value">${initial_positions['joint_1']}</param>
+					</state_interface>
+					<state_interface name="velocity"></state_interface>
+				</joint>
+				<joint name="joint_2">
+					<command_interface name="position"></command_interface>
+					<command_interface name="velocity"></command_interface>
+					<state_interface name="position">
+						<param name="initial_value">${initial_positions['joint_2']}</param>
+					</state_interface>
+					<state_interface name="velocity"></state_interface>
+				</joint>
+				<joint name="joint_3">
+					<command_interface name="position"></command_interface>
+					<command_interface name="velocity"></command_interface>
+					<state_interface name="position">
+						<param name="initial_value">${initial_positions['joint_3']}</param>
+					</state_interface>
+					<state_interface name="velocity"></state_interface>
+				</joint>
+				<joint name="joint_4">
+					<command_interface name="position"></command_interface>
+					<command_interface name="velocity"></command_interface>
+					<state_interface name="position">
+						<param name="initial_value">${initial_positions['joint_4']}</param>
+					</state_interface>
+					<state_interface name="velocity"></state_interface>
+				</joint>
+				<joint name="joint_5">
+					<command_interface name="position"></command_interface>
+					<command_interface name="velocity"></command_interface>
+					<state_interface name="position">
+						<param name="initial_value">${initial_positions['joint_5']}</param>
+					</state_interface>
+					<state_interface name="velocity"></state_interface>
+				</joint>
+				<joint name="joint_6">
+					<command_interface name="position"></command_interface>
+					<command_interface name="velocity"></command_interface>
+					<state_interface name="position">
+						<param name="initial_value">${initial_positions['joint_6']}</param>
+					</state_interface>
+					<state_interface name="velocity"></state_interface>
+				</joint>
+			</ros2_control>
+		</xacro:property>
 	</xacro:macro>
 </robot>
