Commit message: enrich ros2 control node

File: config/i608.ros2_control.xacro (robot description, xacro)
@@ -2,5 +2,59 @@
 <robot xmlns:xacro="http://www.ros.org/wiki/xacro" name="i608">
 	<xacro:macro name="i608_ros2_control" params="name initial_position_file">
-		<xacro:property name="initial_positions" value="${load_yaml(initial_positions_file)['initial_positions']}"></xacro:property>
+		<xacro:property name="initial_positions" value="${load_yaml(initial_positions_file)['initial_positions']}">
+			<ros2_control name="${name}" type="system">
+				<hardware>
+					<plugin>icnc_control_hardware/I608SystemHardware</plugin>
+				</hardware>
+				<joint name="joint_1">
+					<command_interface name="position"></command_interface>
+					<command_interface name="velocity"></command_interface>
+					<state_interface name="position">
+						<param name="initial_value">${initial_positions['joint_1']}</param>
+					</state_interface>
+					<state_interface name="velocity"></state_interface>
+				</joint>
+				<joint name="joint_2">
+					<command_interface name="position"></command_interface>
+					<command_interface name="velocity"></command_interface>
+					<state_interface name="position">
+						<param name="initial_value">${initial_positions['joint_2']}</param>
+					</state_interface>
+					<state_interface name="velocity"></state_interface>
+				</joint>
+				<joint name="joint_3">
+					<command_interface name="position"></command_interface>
+					<command_interface name="velocity"></command_interface>
+					<state_interface name="position">
+						<param name="initial_value">${initial_positions['joint_3']}</param>
+					</state_interface>
+					<state_interface name="velocity"></state_interface>
+				</joint>
+				<joint name="joint_4">
+					<command_interface name="position"></command_interface>
+					<command_interface name="velocity"></command_interface>
+					<state_interface name="position">
+						<param name="initial_value">${initial_positions['joint_4']}</param>
+					</state_interface>
+					<state_interface name="velocity"></state_interface>
+				</joint>
+				<joint name="joint_5">
+					<command_interface name="position"></command_interface>
+					<command_interface name="velocity"></command_interface>
+					<state_interface name="position">
+						<param name="initial_value">${initial_positions['joint_5']}</param>
+					</state_interface>
+					<state_interface name="velocity"></state_interface>
+				</joint>
+				<joint name="joint_6">
+					<command_interface name="position"></command_interface>
+					<command_interface name="velocity"></command_interface>
+					<state_interface name="position">
+						<param name="initial_value">${initial_positions['joint_6']}</param>
+					</state_interface>
+					<state_interface name="velocity"></state_interface>
+				</joint>
+			</ros2_control>
+		</xacro:property>
 	</xacro:macro>
 </robot>

Commit message: Update i608.ros2_control.xacro

File: config/i608.ros2_control.xacro (robot description, xacro)
@@ -2,59 +2,58 @@
 <robot xmlns:xacro="http://www.ros.org/wiki/xacro" name="i608">
 	<xacro:macro name="i608_ros2_control" params="name initial_position_file">
-		<xacro:property name="initial_positions" value="${load_yaml(initial_positions_file)['initial_positions']}">
-			<ros2_control name="${name}" type="system">
-				<hardware>
-					<plugin>icnc_control_hardware/I608SystemHardware</plugin>
-				</hardware>
-				<joint name="joint_1">
-					<command_interface name="position"></command_interface>
-					<command_interface name="velocity"></command_interface>
-					<state_interface name="position">
-						<param name="initial_value">${initial_positions['joint_1']}</param>
-					</state_interface>
-					<state_interface name="velocity"></state_interface>
-				</joint>
-				<joint name="joint_2">
-					<command_interface name="position"></command_interface>
-					<command_interface name="velocity"></command_interface>
-					<state_interface name="position">
-						<param name="initial_value">${initial_positions['joint_2']}</param>
-					</state_interface>
-					<state_interface name="velocity"></state_interface>
-				</joint>
-				<joint name="joint_3">
-					<command_interface name="position"></command_interface>
-					<command_interface name="velocity"></command_interface>
-					<state_interface name="position">
-						<param name="initial_value">${initial_positions['joint_3']}</param>
-					</state_interface>
-					<state_interface name="velocity"></state_interface>
-				</joint>
-				<joint name="joint_4">
-					<command_interface name="position"></command_interface>
-					<command_interface name="velocity"></command_interface>
-					<state_interface name="position">
-						<param name="initial_value">${initial_positions['joint_4']}</param>
-					</state_interface>
-					<state_interface name="velocity"></state_interface>
-				</joint>
-				<joint name="joint_5">
-					<command_interface name="position"></command_interface>
-					<command_interface name="velocity"></command_interface>
-					<state_interface name="position">
-						<param name="initial_value">${initial_positions['joint_5']}</param>
-					</state_interface>
-					<state_interface name="velocity"></state_interface>
-				</joint>
-				<joint name="joint_6">
-					<command_interface name="position"></command_interface>
-					<command_interface name="velocity"></command_interface>
-					<state_interface name="position">
-						<param name="initial_value">${initial_positions['joint_6']}</param>
-					</state_interface>
-					<state_interface name="velocity"></state_interface>
-				</joint>
-			</ros2_control>
-		</xacro:property>
+		<xacro:property name="initial_positions" value="${load_yaml(initial_positions_file)['initial_positions']}"></xacro:property>
+		<ros2_control name="${name}" type="system">
+			<hardware>
+				<plugin>icnc_hardware_interfaces/I608FakeSystemHardware</plugin>
+			</hardware>
+			<joint name="joint_1">
+				<command_interface name="position"></command_interface>
+				<command_interface name="velocity"></command_interface>
+				<state_interface name="position">
+					<param name="initial_value">${initial_positions['joint_1']}</param>
+				</state_interface>
+				<state_interface name="velocity"></state_interface>
+			</joint>
+			<joint name="joint_2">
+				<command_interface name="position"></command_interface>
+				<command_interface name="velocity"></command_interface>
+				<state_interface name="position">
+					<param name="initial_value">${initial_positions['joint_2']}</param>
+				</state_interface>
+				<state_interface name="velocity"></state_interface>
+			</joint>
+			<joint name="joint_3">
+				<command_interface name="position"></command_interface>
+				<command_interface name="velocity"></command_interface>
+				<state_interface name="position">
+					<param name="initial_value">${initial_positions['joint_3']}</param>
+				</state_interface>
+				<state_interface name="velocity"></state_interface>
+			</joint>
+			<joint name="joint_4">
+				<command_interface name="position"></command_interface>
+				<command_interface name="velocity"></command_interface>
+				<state_interface name="position">
+					<param name="initial_value">${initial_positions['joint_4']}</param>
+				</state_interface>
+				<state_interface name="velocity"></state_interface>
+			</joint>
+			<joint name="joint_5">
+				<command_interface name="position"></command_interface>
+				<command_interface name="velocity"></command_interface>
+				<state_interface name="position">
+					<param name="initial_value">${initial_positions['joint_5']}</param>
+				</state_interface>
+				<state_interface name="velocity"></state_interface>
+			</joint>
+			<joint name="joint_6">
+				<command_interface name="position"></command_interface>
+				<command_interface name="velocity"></command_interface>
+				<state_interface name="position">
+					<param name="initial_value">${initial_positions['joint_6']}</param>
+				</state_interface>
+				<state_interface name="velocity"></state_interface>
+			</joint>
+		</ros2_control>
 	</xacro:macro>
 </robot>

Commit message: Update i608.ros2_control.xacro

File: config/i608.ros2_control.xacro (robot description, xacro)
@@ -1,5 +1,5 @@
 <?xml version="1.0"?>
 <robot xmlns:xacro="http://www.ros.org/wiki/xacro" name="i608">
-	<xacro:macro name="i608_ros2_control" params="name initial_position_file">
+	<xacro:macro name="i608_ros2_control" params="name initial_positions_file">
 		<xacro:property name="initial_positions" value="${load_yaml(initial_positions_file)['initial_positions']}"></xacro:property>
 		<ros2_control name="${name}" type="system">

Commit message: rm initial_positions

File: config/i608.ros2_control.xacro (robot description, xacro)
@@ -1,6 +1,7 @@
 <?xml version="1.0"?>
 <robot xmlns:xacro="http://www.ros.org/wiki/xacro" name="i608">
-	<xacro:macro name="i608_ros2_control" params="name initial_positions_file">
-		<xacro:property name="initial_positions" value="${load_yaml(initial_positions_file)['initial_positions']}"></xacro:property>
+	<!-- params="name initial_positions_file" -->
+	<xacro:macro name="i608_ros2_control">
+		<!-- <xacro:property name="initial_positions" value="${load_yaml(initial_positions_file)['initial_positions']}"></xacro:property> -->
 		<ros2_control name="${name}" type="system">
 			<hardware>
@@ -11,5 +12,5 @@
 				<command_interface name="velocity"></command_interface>
 				<state_interface name="position">
-					<param name="initial_value">${initial_positions['joint_1']}</param>
+					<!-- <param name="initial_value">${initial_positions['joint_1']}</param> -->
 				</state_interface>
 				<state_interface name="velocity"></state_interface>
@@ -19,5 +20,5 @@
 				<command_interface name="velocity"></command_interface>
 				<state_interface name="position">
-					<param name="initial_value">${initial_positions['joint_2']}</param>
+					<!-- <param name="initial_value">${initial_positions['joint_2']}</param> -->
 				</state_interface>
 				<state_interface name="velocity"></state_interface>
@@ -27,5 +28,5 @@
 				<command_interface name="velocity"></command_interface>
 				<state_interface name="position">
-					<param name="initial_value">${initial_positions['joint_3']}</param>
+					<!-- <param name="initial_value">${initial_positions['joint_3']}</param> -->
 				</state_interface>
 				<state_interface name="velocity"></state_interface>
@@ -35,5 +36,5 @@
 				<command_interface name="velocity"></command_interface>
 				<state_interface name="position">
-					<param name="initial_value">${initial_positions['joint_4']}</param>
+					<!-- <param name="initial_value">${initial_positions['joint_4']}</param> -->
 				</state_interface>
 				<state_interface name="velocity"></state_interface>
@@ -43,5 +44,5 @@
 				<command_interface name="velocity"></command_interface>
 				<state_interface name="position">
-					<param name="initial_value">${initial_positions['joint_5']}</param>
+					<!-- <param name="initial_value">${initial_positions['joint_5']}</param> -->
 				</state_interface>
 				<state_interface name="velocity"></state_interface>
@@ -51,5 +52,5 @@
 				<command_interface name="velocity"></command_interface>
 				<state_interface name="position">
-					<param name="initial_value">${initial_positions['joint_6']}</param>
+					<!-- <param name="initial_value">${initial_positions['joint_6']}</param> -->
 				</state_interface>
 				<state_interface name="velocity"></state_interface>

File: config/i608.urdf.xacro (robot description, xacro)
@@ -1,7 +1,8 @@
 <?xml version="1.0"?>
 <robot xmlns:xacro="http://www.ros.org/wiki/xacro" name="i608">
-	<xacro:arg name="initial_positions_file" default="initial_positions.yaml" />
+	<!-- <xacro:arg name="initial_positions_file" default="initial_positions.yaml" /> -->
 	<xacro:include filename="$(find icnc_resources_i608_description)/urdf/i608.urdf" />
 	<xacro:include filename="i608.ros2_control.xacro" />
-	<xacro:i608_ros2_control name="I608SystemPV" initial_positions_file="$(arg initial_positions_file)" />
+	<!-- initial_positions_file="$(arg initial_positions_file)" -->
+	<xacro:i608_ros2_control name="I608SystemPV" />
 </robot>

Commit message: rm initial_positions

File: config/i608.ros2_control.xacro (robot description, xacro)
@@ -1,8 +1,6 @@
 <?xml version="1.0"?>
 <robot xmlns:xacro="http://www.ros.org/wiki/xacro" name="i608">
-	<!-- params="name initial_positions_file" -->
 	<xacro:macro name="i608_ros2_control">
-		<!-- <xacro:property name="initial_positions" value="${load_yaml(initial_positions_file)['initial_positions']}"></xacro:property> -->
-		<ros2_control name="${name}" type="system">
+		<ros2_control type="system">
 			<hardware>
 				<plugin>icnc_fake_hardware_interfaces/I608FakeHardwareInterface</plugin>
@@ -11,7 +9,5 @@
 				<command_interface name="position"></command_interface>
 				<command_interface name="velocity"></command_interface>
-				<state_interface name="position">
-					<!-- <param name="initial_value">${initial_positions['joint_1']}</param> -->
-				</state_interface>
+				<state_interface name="position"></state_interface>
 				<state_interface name="velocity"></state_interface>
 			</joint>
@@ -19,7 +15,5 @@
 				<command_interface name="position"></command_interface>
 				<command_interface name="velocity"></command_interface>
-				<state_interface name="position">
-					<!-- <param name="initial_value">${initial_positions['joint_2']}</param> -->
-				</state_interface>
+				<state_interface name="position"></state_interface>
 				<state_interface name="velocity"></state_interface>
 			</joint>
@@ -27,7 +21,5 @@
 				<command_interface name="position"></command_interface>
 				<command_interface name="velocity"></command_interface>
-				<state_interface name="position">
-					<!-- <param name="initial_value">${initial_positions['joint_3']}</param> -->
-				</state_interface>
+				<state_interface name="position"></state_interface>
 				<state_interface name="velocity"></state_interface>
 			</joint>
@@ -35,7 +27,5 @@
 				<command_interface name="position"></command_interface>
 				<command_interface name="velocity"></command_interface>
-				<state_interface name="position">
-					<!-- <param name="initial_value">${initial_positions['joint_4']}</param> -->
-				</state_interface>
+				<state_interface name="position"></state_interface>
 				<state_interface name="velocity"></state_interface>
 			</joint>
@@ -43,7 +33,5 @@
 				<command_interface name="position"></command_interface>
 				<command_interface name="velocity"></command_interface>
-				<state_interface name="position">
-					<!-- <param name="initial_value">${initial_positions['joint_5']}</param> -->
-				</state_interface>
+				<state_interface name="position"></state_interface>
 				<state_interface name="velocity"></state_interface>
 			</joint>
@@ -51,7 +39,5 @@
 				<command_interface name="position"></command_interface>
 				<command_interface name="velocity"></command_interface>
-				<state_interface name="position">
-					<!-- <param name="initial_value">${initial_positions['joint_6']}</param> -->
-				</state_interface>
+				<state_interface name="position"></state_interface>
 				<state_interface name="velocity"></state_interface>
 			</joint>

File: config/i608.urdf.xacro (robot description, xacro)
@@ -1,8 +1,6 @@
 <?xml version="1.0"?>
 <robot xmlns:xacro="http://www.ros.org/wiki/xacro" name="i608">
-	<!-- <xacro:arg name="initial_positions_file" default="initial_positions.yaml" /> -->
 	<xacro:include filename="$(find icnc_resources_i608_description)/urdf/i608.urdf" />
 	<xacro:include filename="i608.ros2_control.xacro" />
-	<!-- initial_positions_file="$(arg initial_positions_file)" -->
 	<xacro:i608_ros2_control name="I608SystemPV" />
 </robot>

Commit message: Update i608.ros2_control.xacro

File: config/i608.ros2_control.xacro (robot description, xacro)
@@ -1,44 +1,44 @@
 <?xml version="1.0"?>
 <robot xmlns:xacro="http://www.ros.org/wiki/xacro" name="i608">
-	<xacro:macro name="i608_ros2_control">
-		<ros2_control type="system">
+	<xacro:macro name="i608_ros2_control" params="name">
+		<ros2_control name="${name}" type="system">
 			<hardware>
 				<plugin>icnc_fake_hardware_interfaces/I608FakeHardwareInterface</plugin>
 			</hardware>
 			<joint name="joint_1">
-				<command_interface name="position"></command_interface>
-				<command_interface name="velocity"></command_interface>
-				<state_interface name="position"></state_interface>
-				<state_interface name="velocity"></state_interface>
+				<command_interface name="position" />
+				<command_interface name="velocity" />
+				<state_interface name="position" />
+				<state_interface name="velocity" />
 			</joint>
 			<joint name="joint_2">
-				<command_interface name="position"></command_interface>
-				<command_interface name="velocity"></command_interface>
-				<state_interface name="position"></state_interface>
-				<state_interface name="velocity"></state_interface>
+				<command_interface name="position" />
+				<command_interface name="velocity" />
+				<state_interface name="position" />
+				<state_interface name="velocity" />
 			</joint>
 			<joint name="joint_3">
-				<command_interface name="position"></command_interface>
-				<command_interface name="velocity"></command_interface>
-				<state_interface name="position"></state_interface>
-				<state_interface name="velocity"></state_interface>
+				<command_interface name="position" />
+				<command_interface name="velocity" />
+				<state_interface name="position" />
+				<state_interface name="velocity" />
 			</joint>
 			<joint name="joint_4">
-				<command_interface name="position"></command_interface>
-				<command_interface name="velocity"></command_interface>
-				<state_interface name="position"></state_interface>
-				<state_interface name="velocity"></state_interface>
+				<command_interface name="position" />
+				<command_interface name="velocity" />
+				<state_interface name="position" />
+				<state_interface name="velocity" />
 			</joint>
 			<joint name="joint_5">
-				<command_interface name="position"></command_interface>
-				<command_interface name="velocity"></command_interface>
-				<state_interface name="position"></state_interface>
-				<state_interface name="velocity"></state_interface>
+				<command_interface name="position" />
+				<command_interface name="velocity" />
+				<state_interface name="position" />
+				<state_interface name="velocity" />
 			</joint>
 			<joint name="joint_6">
-				<command_interface name="position"></command_interface>
-				<command_interface name="velocity"></command_interface>
-				<state_interface name="position"></state_interface>
-				<state_interface name="velocity"></state_interface>
+				<command_interface name="position" />
+				<command_interface name="velocity" />
+				<state_interface name="position" />
+				<state_interface name="velocity" />
 			</joint>
 		</ros2_control>
