Commit message: check

File: panda_moveit_config/config/panda_hand.ros2_control.xacro (robot description, xacro)
@@ -1,26 +1,26 @@
 <?xml version="1.0"?>
 <robot xmlns:xacro="http://www.ros.org/wiki/xacro">
-	<xacro:macro name="panda_hand_ros2_control" params="name">
-		<ros2_control name="${name}" type="system">
-			<hardware>
-				<plugin>mock_components/GenericSystem</plugin>
-			</hardware>
-			<joint name="panda_finger_joint1">
-				<command_interface name="poisition"/>
-				<state_interface name="position">
-					<param name="initial_value">0.0</param>
-				</state_interface>
-				<state_interface name="velocity"/>
-			</joint>
-			<joint name="panda_finger_joint1">
-				<param name="mimic">panda_finger_joint1</param>
-				<param name="multiplier">1</param>
-				<command_interface name="position"/>
-				<state_interface name="position">
-					<param name="initial_value">0.0</param>
-				</state_interface>
-				<state_interface name="velocity"/>
-			</joint>
-		</ros2_control>
-	</xacro:macro>
+    <xacro:macro name="panda_hand_ros2_control" params="name">
+        <ros2_control name="${name}" type="system">
+            <hardware>
+                <plugin>mock_components/GenericSystem</plugin>
+            </hardware>
+            <joint name="panda_finger_joint1">
+                <command_interface name="position" />
+                <state_interface name="position">
+                  <param name="initial_value">0.0</param>
+                </state_interface>
+                <state_interface name="velocity"/>
+            </joint>
+            <joint name="panda_finger_joint2">
+                <param name="mimic">panda_finger_joint1</param>
+                <param name="multiplier">1</param>
+                <command_interface name="position" />
+                <state_interface name="position">
+                  <param name="initial_value">0.0</param>
+                </state_interface>
+                <state_interface name="velocity"/>
+            </joint>
+        </ros2_control>
+    </xacro:macro>
 </robot>
